Commit message: corrected wheel's rotation direction

File: ros2_ws/src/ssl_robot/urdf/robot.urdf (robot description, URDF)
Before this commit: robot robot, 6 links, 5 joints
Links:
- link link_BR: mass 0.0331917400647206 -> 0.0331917384702334
- link link_FL: mass 0.0331917384702334 -> 0.0331917400647206
Joints:
- joint joint_BL: axis 0 1 0 -> 0 -1 0; origin xyz=0.0285 0.09 -0.06 rpy=0 0 0 -> xyz=0.028512 0.046531 -0.08294 rpy=1.569003673 2.598396327 1.5708
- joint joint_BR: origin xyz=0.0285 -0.09 -0.06 rpy=0 0 0 -> xyz=0.028512 -0.092037 -0.04871 rpy=-1.571882827 -1.027516327 -1.5708
- joint joint_FL: origin xyz=0.0285 0.09 0.06 rpy=0 0 0 -> xyz=0.028512 0.091331 0.03148 rpy=-1.570203673 1.289446327 1.5708
- joint joint_FR: axis 0 1 0 -> 0 -1 0; origin xyz=0.0285 -0.09 0.06 rpy=0 0 0 -> xyz=0.028512 -0.078256 0.073565 rpy=1.572253127 -2.336636327 -1.5708

Commit message: Increased obot size

File: ros2_ws/src/ssl_robot/urdf/robot.urdf (robot description, URDF)
Before this commit: robot robot, 6 links, 5 joints
Links:
- link base_link: mass 0.643917957153286 -> 41.2097288570119; geometry collision mesh filename=package://ssl_robot/meshes/base_link.STL scale=4 4 4; visual mesh filename=package://ssl_robot/meshes/base_link.STL scale=4 4 4
- link link_BL: mass 0.0331917385997145 -> 2.12437447038128; geometry collision mesh filename=package://ssl_robot/meshes/link_BL.STL scale=4 4 4; visual mesh filename=package://ssl_robot/meshes/link_BL.STL scale=4 4 4
- link link_BR: mass 0.0331917400647206 -> 2.1243737652629; geometry collision mesh filename=package://ssl_robot/meshes/link_BR.STL scale=4 4 4; visual mesh filename=package://ssl_robot/meshes/link_BR.STL scale=4 4 4
- link link_FL: mass 0.0331917384702334 -> 2.12437444606277; geometry collision mesh filename=package://ssl_robot/meshes/link_FL.STL scale=4 4 4; visual mesh filename=package://ssl_robot/meshes/link_FL.STL scale=4 4 4
- link link_FR: mass 0.0331917386699706 -> 2.12437439391811; geometry collision mesh filename=package://ssl_robot/meshes/link_FR.STL scale=4 4 4; visual mesh filename=package://ssl_robot/meshes/link_FR.STL scale=4 4 4
Joints:
- joint joint_BL: origin xyz=0.0285 0.09 -0.06 rpy=0 0 0 -> xyz=0.114 0.36 -0.24 rpy=0 0 0
- joint joint_BR: origin xyz=0.0285 -0.09 -0.06 rpy=0 0 0 -> xyz=0.114  -0.36  -0.24 rpy=0 0 0
- joint joint_FL: origin xyz=0.0285 0.09 0.06 rpy=0 0 0 -> xyz=0.114 0.36 0.24 rpy=0 0 0
- joint joint_FR: origin xyz=0.0285 -0.09 0.06 rpy=0 0 0 -> xyz=0.114 -0.36 0.24 rpy=0 0 0

Commit message: merging U.R and H_A

File: ros2_ws/src/ssl_robot/urdf/robot.urdf (robot description, URDF)
Before this commit: robot robot, 6 links, 5 joints
Links:
- link base_link: mass 0.643917957153286 -> 41.2097288570119; geometry collision mesh filename=package://ssl_robot/meshes/base_link.STL scale=4 4 4; visual mesh filename=package://ssl_robot/meshes/base_link.STL scale=4 4 4
- link link_BL: mass 0.0331917385997145 -> 2.12437447038128; geometry collision mesh filename=package://ssl_robot/meshes/link_BL.STL scale=4 4 4; visual mesh filename=package://ssl_robot/meshes/link_BL.STL scale=4 4 4
- link link_BR: mass 0.0331917384702334 -> 2.1243737652629; geometry collision mesh filename=package://ssl_robot/meshes/link_BR.STL scale=4 4 4; visual mesh filename=package://ssl_robot/meshes/link_BR.STL scale=4 4 4
- link link_FL: mass 0.0331917400647206 -> 2.12437444606277; geometry collision mesh filename=package://ssl_robot/meshes/link_FL.STL scale=4 4 4; visual mesh filename=package://ssl_robot/meshes/link_FL.STL scale=4 4 4
- link link_FR: mass 0.0331917386699706 -> 2.12437439391811; geometry collision mesh filename=package://ssl_robot/meshes/link_FR.STL scale=4 4 4; visual mesh filename=package://ssl_robot/meshes/link_FR.STL scale=4 4 4
Joints:
- joint joint_BL: axis 0 -1 0 -> 0 1 0; origin xyz=0.028512 0.046531 -0.08294 rpy=1.569003673 2.598396327 1.5708 -> xyz=0.114 0.36 -0.24 rpy=0 0 0
- joint joint_BR: origin xyz=0.028512 -0.092037 -0.04871 rpy=-1.571882827 -1.027516327 -1.5708 -> xyz=0.114  -0.36  -0.24 rpy=0 0 0
- joint joint_FL: origin xyz=0.028512 0.091331 0.03148 rpy=-1.570203673 1.289446327 1.5708 -> xyz=0.114 0.36 0.24 rpy=0 0 0
- joint joint_FR: axis 0 -1 0 -> 0 1 0; origin xyz=0.028512 -0.078256 0.073565 rpy=1.572253127 -2.336636327 -1.5708 -> xyz=0.114 -0.36 0.24 rpy=0 0 0

Commit message: Update robot.urdf
fixed a small bug

File: ros2_ws/src/ssl_robot/urdf/robot.urdf (robot description, URDF)
Before this commit: robot robot_scaled, 6 links, 5 joints
Joints:
- joint joint_BL: axis 0 1 0 -> 0 -1 0; origin xyz=0.114 0.36 -0.24 rpy=0 0 0 -> xyz=0.114048 0.186124 -0.33176 rpy=1.569003673 2.598396327 1.5708
- joint joint_BR: axis 0 1 0 -> 0 -1 0; origin xyz=0.114  -0.36  -0.24 rpy=0 0 0 -> xyz=0.11404 -0.368148 -0.19484 rpy=-1.571882827 2.114076334 -1.5708
- joint joint_FL: axis 0 1 0 -> 0 -1 0; origin xyz=0.114 0.36 0.24 rpy=0 0 0 -> xyz=0.114048 0.365324 0.12592 rpy=-1.570203673 4.431038981 1.5708
- joint joint_FR: axis 0 1 0 -> 0 -1 0; origin xyz=0.114 -0.36 0.24 rpy=0 0 0 -> xyz=0.114048 -0.313024 0.29426 rpy=1.572253127 -2.336636327 -1.5708
